File: Schematic/RPM411/RPM411.kicad_pcb (KiCad board)
At the start: 2 copper layers, 74 parts, among them U1 STM32F100C8Tb8

Commit message: added pressure cap
Parts:
- added P1: P_Cap, RPM411:Pressure_Cap, F.Cu at (81.3, 93.9)
- added R34: DNP, Resistor_SMD:R_0402_1005Metric, F.Cu at (94.0, 78.7)
Changed lines of the file:
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@@
   (net 193 "unconnected-(R33-Pad1)")
   (net 194 "unconnected-(R33-Pad2)")
+  (net 195 "unconnected-(P1-Pad1)")
+  (net 196 "unconnected-(P1-Pad2)")
+  (net 197 "unconnected-(P1-PadSH)")
+  (net 198 "unconnected-(R34-Pad1)")
+  (net 199 "unconnected-(R34-Pad2)")
   (footprint "Capacitor_SMD:C_0402_1005Metric" (layer "F.Cu")
     (at 99.43 69.68)
@@
     )
   )
+  (footprint "RPM411:Pressure_Cap" (layer "F.Cu")
+    (at 81.28 93.9275)
+    (property "Sheetfile" "RPM411.kicad_sch")
+    (property "Sheetname" "")
+    (attr smd)
+    (fp_text reference "P1" (at 0 2.54 unlocked) (layer "F.SilkS")
+      (effects (font (size 1 1) (thickness 0.15)))
+    )
+    (fp_text value "P_Cap" (at 0 -3.81 unlocked) (layer "F.Fab")
+      (effects (font (size 1 1) (thickness 0.15)))
+    )
+    (fp_text user "${REFERENCE}" (at 0 -2.54 unlocked) (layer "F.Fab")
+      (effects (font (size 1 1) (thickness 0.15)))
+    )
+    (fp_line (start 5.08 -0.635) (end 5.08 -10.795) (layer "F.SilkS") (width 0.12))
+    (fp_line (start 0 -0.635) (end 5.08 -0.635) (layer "F.SilkS") (width 0.12))
+    (fp_line (start -5.08 -0.635) (end 0 -0.635) (layer "F.SilkS") (width 0.12))
+    (fp_line (start 5.08 -10.795) (end -5.08 -10.795) (layer "F.SilkS") (width 0.12))
+    (fp_line (start -5.08 -10.795) (end -5.08 -0.635) (layer "F.SilkS") (width 0.12))
+    (fp_rect (start -0.635 -8.255) (end 1.905 -5.715) (layer "F.SilkS") (width 0.12) (fill none))
+    (fp_circle (center 0 -5.715) (end 4.445 -5.715) (layer "F.SilkS") (width 0.12) (fill none))
+    (fp_line (start 0 0) (end 5.715 0) (layer "F.CrtYd") (width 0.05))
+    (fp_line (start -5.715 -11.43) (end -5.715 0) (layer "F.CrtYd") (width 0.05))
+    (fp_line (start 5.715 -11.43) (end -5.715 -11.43) (layer "F.CrtYd") (width 0.05))
+    (fp_line (start 5.715 0) (end 5.715 -11.43) (layer "F.CrtYd") (width 0.05))
+    (fp_line (start -5.715 0) (end 0 0) (layer "F.CrtYd") (width 0.05))
+    (pad "1" smd rect (at -3.175 0) (size 1.5 2.8) (layers "F.Cu" "F.Paste" "F.Mask")
+      (net 195 "unconnected-(P1-Pad1)") (pintype "passive"))
+    (pad "2" smd rect (at 3.175 0) (size 1.5 2.8) (layers "F.Cu" "F.Paste" "F.Mask")
+      (net 196 "unconnected-(P1-Pad2)") (pintype "passive"))
+    (pad "SH" smd rect (at 0 0) (size 1.5 2.8) (layers "F.Cu" "F.Paste" "F.Mask")
+      (net 197 "unconnected-(P1-PadSH)") (pinfunction "SH") (pintype "passive"))
+  )
   (footprint "Inductor_SMD:L_0402_1005Metric" (layer "F.Cu")
     (at 79.16 71.72)
@@
     (model "${KICAD6_3DMODEL_DIR}/Resistor_SMD.3dshapes/R_0402_1005Metric.wrl"
       (offset (xyz 0 0 0))
+      (scale (xyz 1 1 1))
+      (rotate (xyz 0 0 0))
+    )
+  )
+  (footprint "Resistor_SMD:R_0402_1005Metric" (layer "F.Cu")
+    (at 93.98 78.74)
+    (descr "Resistor SMD 0402 (1005 Metric), square (rectangular) end terminal, IPC_7351 nominal, (Body size source: IPC-SM-782 page 72, https://www.pcb-3d.com/wordpress/wp-content/uploads/ipc-sm-782a_amendment_1_and_2.pdf), generated with kicad-footprint-generator")
+    (tags "resistor")
+    (property "Sheetfile" "RPM411.kicad_sch")
+    (property "Sheetname" "")
+    (attr smd)
+    (fp_text reference "R34" (at 0 -1.17) (layer "F.SilkS")
+      (effects (font (size 1 1) (thickness 0.15)))
+    )
+    (fp_text value "DNP" (at 0 1.17) (layer "F.Fab")
+      (effects (font (size 1 1) (thickness 0.15)))
+    )
+    (fp_text user "${REFERENCE}" (at 0 0) (layer "F.Fab")
+      (effects (font (size 0.26 0.26) (thickness 0.04)))
+    )
+    (fp_line (start -0.153641 -0.38) (end 0.153641 -0.38) (layer "F.SilkS") (width 0.12))
+    (fp_line (start -0.153641 0.38) (end 0.153641 0.38) (layer "F.SilkS") (width 0.12))
+    (fp_line (start -0.93 0.47) (end -0.93 -0.47) (layer "F.CrtYd") (width 0.05))
+    (fp_line (start 0.93 -0.47) (end 0.93 0.47) (layer "F.CrtYd") (width 0.05))
+    (fp_line (start -0.93 -0.47) (end 0.93 -0.47) (layer "F.CrtYd") (width 0.05))
+    (fp_line (start 0.93 0.47) (end -0.93 0.47) (layer "F.CrtYd") (width 0.05))
+    (fp_line (start 0.525 -0.27) (end 0.525 0.27) (layer "F.Fab") (width 0.1))
+    (fp_line (start -0.525 0.27) (end -0.525 -0.27) (layer "F.Fab") (width 0.1))
+    (fp_line (start -0.525 -0.27) (end 0.525 -0.27) (layer "F.Fab") (width 0.1))
+    (fp_line (start 0.525 0.27) (end -0.525 0.27) (layer "F.Fab") (width 0.1))
+    (pad "1" smd roundrect (at -0.51 0) (size 0.54 0.64) (layers "F.Cu" "F.Paste" "F.Mask") (roundrect_rratio 0.25)
+      (net 198 "unconnected-(R34-Pad1)") (pintype "passive"))
+    (pad "2" smd roundrect (at 0.51 0) (size 0.54 0.64) (layers "F.Cu" "F.Paste" "F.Mask") (roundrect_rratio 0.25)
+      (net 199 "unconnected-(R34-Pad2)") (pintype "passive"))
+    (model "${KICAD6_3DMODEL_DIR}/Resistor_SMD.3dshapes/R_0402_1005Metric.wrl"
+      (offset (xyz 0 0 0))

Commit message: identified ICs
Parts:
- added Q1: tbd (GDS), Package_TO_SOT_SMD:SOT-523, F.Cu at (101.6, 88.9)
- added U2: TS5A9411, Package_TO_SOT_SMD:SOT-363_SC-70-6, F.Cu at (91.4, 94.0)
- added U3: TS5A9411, Package_TO_SOT_SMD:SOT-363_SC-70-6, F.Cu at (91.4, 99.1)
- added U4: TS5A9411, Package_TO_SOT_SMD:SOT-363_SC-70-6, F.Cu at (99.9, 99.1)
- added U5: 74LVC3G04, Package_SO:SSOP-8_3.95x5.21x3.27mm_P1.27mm, F.Cu at (91.5, 86.3)
- added U6: 74LVC1G32, Package_TO_SOT_SMD:SOT-353_SC-70-5, F.Cu at (95.7, 99.1)
- added U7: TLV70030DDC, Package_TO_SOT_SMD:SOT-23-5, F.Cu at (98.2, 85.1)

Commit message: completed schematic
Parts:
- added J1: 02x08_tbd, Connector_PinHeader_1.00mm:PinHeader_2x08_P1.00mm_Vertical, F.Cu at (104.1, 73.7)
- added TP1: Pin5, TestPoint:TestPoint_Pad_D1.0mm, F.Cu at (134.6, 68.6)
- added TP2: CS_E, TestPoint:TestPoint_Pad_D1.0mm, F.Cu at (134.6, 71.6)
- added TP3: CS_P, TestPoint:TestPoint_Pad_D1.0mm, F.Cu at (131.6, 71.6)
- added TP4: SDI, TestPoint:TestPoint_Pad_D1.0mm, F.Cu at (131.6, 68.6)
Connections:
- C1 pad 1: unconnected-(C1-Pad1) -> +3V8
- C1 pad 2: unconnected-(C1-Pad2) -> GND
- C10 pad 1: unconnected-(C10-Pad1) -> VDD
- C10 pad 2: unconnected-(C10-Pad2) -> GND
- C11 pad 1: unconnected-(C11-Pad1) -> LED
- C11 pad 2: unconnected-(C11-Pad2) -> GND
- C12 pad 1: unconnected-(C12-Pad1) -> GND
- C12 pad 2: unconnected-(C12-Pad2) -> Pullup
- C13 pad 1: unconnected-(C13-Pad1) -> VDD
- C13 pad 2: unconnected-(C13-Pad2) -> GND
- C14 pad 1: unconnected-(C14-Pad1) -> Switch_1
- C14 pad 2: unconnected-(C14-Pad2) -> GND
- C15 pad 1: unconnected-(C15-Pad1) -> Switch_2
- C15 pad 2: unconnected-(C15-Pad2) -> GND
- C16 pad 1: unconnected-(C16-Pad1) -> Switch_3
- C16 pad 2: unconnected-(C16-Pad2) -> GND
- C17 pad 1: unconnected-(C17-Pad1) -> VDD
- C17 pad 2: unconnected-(C17-Pad2) -> GND
- C18 pad 1: unconnected-(C18-Pad1) -> VCC
- C18 pad 2: unconnected-(C18-Pad2) -> GND
- C19 pad 1: unconnected-(C19-Pad1) -> Net-(C33-Pad2)
- C19 pad 2: unconnected-(C19-Pad2) -> Net-(U4-Pad6)
- C2 pad 1: unconnected-(C2-Pad1) -> +3V8
- C2 pad 2: unconnected-(C2-Pad2) -> GND
- C20 pad 1: unconnected-(C20-Pad1) -> VCC
- C20 pad 2: unconnected-(C20-Pad2) -> GND
- C21 pad 1: unconnected-(C21-Pad1) -> VCC
- C21 pad 2: unconnected-(C21-Pad2) -> GND
- C22 pad 1: unconnected-(C22-Pad1) -> VCC
- C22 pad 2: unconnected-(C22-Pad2) -> GND
- C23 pad 1: unconnected-(C23-Pad1) -> Net-(C23-Pad1)
- C23 pad 2: unconnected-(C23-Pad2) -> Net-(U4-Pad6)
- C24 pad 1: unconnected-(C24-Pad1) -> Net-(U6-Pad1)
- C24 pad 2: unconnected-(C24-Pad2) -> GND
- C25 pad 1: unconnected-(C25-Pad1) -> VCC
- C25 pad 2: unconnected-(C25-Pad2) -> GND
- C26 pad 1: unconnected-(C26-Pad1) -> Net-(C33-Pad2)
- C26 pad 2: unconnected-(C26-Pad2) -> Net-(R31-Pad1)
- C27 pad 1: unconnected-(C27-Pad1) -> Net-(U7-Pad5)
- C27 pad 2: unconnected-(C27-Pad2) -> GND
- C28 pad 1: unconnected-(C28-Pad1) -> Net-(U7-Pad5)
- C28 pad 2: unconnected-(C28-Pad2) -> GND
- C29 pad 1: unconnected-(C29-Pad1) -> VCCD_mon
- C29 pad 2: unconnected-(C29-Pad2) -> GND
- C3 pad 1: unconnected-(C3-Pad1) -> VDD
- C3 pad 2: unconnected-(C3-Pad2) -> GND
- C30 pad 1: unconnected-(C30-Pad1) -> Net-(U7-Pad4)
- C30 pad 2: unconnected-(C30-Pad2) -> GND
- C31 pad 1: unconnected-(C31-Pad1) -> +3V8
- C31 pad 2: unconnected-(C31-Pad2) -> GND
- C32 pad 1: unconnected-(C32-Pad1) -> +3V8
- C32 pad 2: unconnected-(C32-Pad2) -> GND
- C33 pad 1: unconnected-(C33-Pad1) -> Net-(U4-Pad5)
- C33 pad 2: unconnected-(C33-Pad2) -> Net-(C33-Pad2)
- C33 pad SH: unconnected-(C33-PadSH) -> GND
- C34 pad 1: unconnected-(C34-Pad1) -> VDD
- C34 pad 2: unconnected-(C34-Pad2) -> GND
- C4 pad 1: unconnected-(C4-Pad1) -> VDD
- C4 pad 2: unconnected-(C4-Pad2) -> GND
- C5 pad 1: unconnected-(C5-Pad1) -> VDD
- C5 pad 2: unconnected-(C5-Pad2) -> GND
- C6 pad 1: unconnected-(C6-Pad1) -> NRST
- C6 pad 2: unconnected-(C6-Pad2) -> GND
- C7 pad 1: unconnected-(C7-Pad1) -> VDD
- C7 pad 2: unconnected-(C7-Pad2) -> GND
- C8 pad 1: unconnected-(C8-Pad1) -> VDD
- C8 pad 2: unconnected-(C8-Pad2) -> GND
- C9 pad 1: unconnected-(C9-Pad1) -> GND
- C9 pad 2: unconnected-(C9-Pad2) -> VCCA_mon
- D1 pad 1: unconnected-(D1-Pad1) -> LED
- D1 pad 2: unconnected-(D1-Pad2) -> Net-(D1-Pad2)
- L1 pad 1: unconnected-(L1-Pad1) -> Net-(J1-Pad2)
- L1 pad 2: unconnected-(L1-Pad2) -> VDD
- L2 pad 1: unconnected-(L2-Pad1) -> GND
- L2 pad 2: unconnected-(L2-Pad2) -> Out
- L3 pad 1: unconnected-(L3-Pad1) -> Net-(U1-Pad22)
- L3 pad 2: unconnected-(L3-Pad2) -> LED
- L4 pad 1: unconnected-(L4-Pad1) -> VCC
- L4 pad 2: unconnected-(L4-Pad2) -> Net-(U7-Pad5)
- P1 pad 1: unconnected-(P1-Pad1) -> Net-(U2-Pad5)
- P1 pad 2: unconnected-(P1-Pad2) -> Net-(C33-Pad2)
- P1 pad SH: unconnected-(P1-PadSH) -> GND
- Q1 pad 1: unconnected-(Q1-Pad1) -> Pullup
- Q1 pad 2: unconnected-(Q1-Pad2) -> VCC
- Q1 pad 3: unconnected-(Q1-Pad3) -> Net-(C33-Pad2)
- R1 pad 1: unconnected-(R1-Pad1) -> Net-(J1-Pad15)
- R1 pad 2: unconnected-(R1-Pad2) -> +3V8
- R10 pad 1: unconnected-(R10-Pad1) -> VCCA_mon
- R10 pad 2: unconnected-(R10-Pad2) -> VCC
- R11 pad 1: unconnected-(R11-Pad1) -> Net-(U1-Pad17)
- R11 pad 2: unconnected-(R11-Pad2) -> SPI_SDI
- R12 pad 1: unconnected-(R12-Pad1) -> Net-(U1-Pad16)
- R12 pad 2: unconnected-(R12-Pad2) -> SPI_SDO
- R13 pad 1: unconnected-(R13-Pad1) -> Net-(U1-Pad15)
- R13 pad 2: unconnected-(R13-Pad2) -> SPI_SCK
- R14 pad 1: unconnected-(R14-Pad1) -> VCCD_mon
- R14 pad 2: unconnected-(R14-Pad2) -> Net-(R14-Pad2)
- R15 pad 1: unconnected-(R15-Pad1) -> Pullup
- R15 pad 2: unconnected-(R15-Pad2) -> Net-(U1-Pad25)
- R16 pad 1: unconnected-(R16-Pad1) -> VDD
- R16 pad 2: unconnected-(R16-Pad2) -> Net-(D1-Pad2)
- R17 pad 1: unconnected-(R17-Pad1) -> Switch_1
- R17 pad 2: unconnected-(R17-Pad2) -> Net-(U1-Pad42)
- R18 pad 1: unconnected-(R18-Pad1) -> Switch_2
- R18 pad 2: unconnected-(R18-Pad2) -> Net-(U1-Pad41)
- R19 pad 1: unconnected-(R19-Pad1) -> Net-(U1-Pad37)
- R19 pad 2: unconnected-(R19-Pad2) -> SWCLK 
- R2 pad 1: unconnected-(R2-Pad1) -> NRST
- R2 pad 2: unconnected-(R2-Pad2) -> Net-(J1-Pad13)
- R20 pad 1: unconnected-(R20-Pad1) -> Switch_3
- R20 pad 2: unconnected-(R20-Pad2) -> Net-(R20-Pad2)
- R21 pad 1: unconnected-(R21-Pad1) -> Net-(U1-Pad34)
- R21 pad 2: unconnected-(R21-Pad2) -> SWDIO
- R22 pad 1: unconnected-(R22-Pad1) -> Net-(U1-Pad30)
- R22 pad 2: unconnected-(R22-Pad2) -> UART_TX
- R23 pad 1: unconnected-(R23-Pad1) -> GND
- R23 pad 2: unconnected-(R23-Pad2) -> GND
- R24 pad 1: unconnected-(R24-Pad1) -> GND
- R24 pad 2: unconnected-(R24-Pad2) -> GND
- R25 pad 1: unconnected-(R25-Pad1) -> GND
- R25 pad 2: unconnected-(R25-Pad2) -> GND
- R26 pad 1: unconnected-(R26-Pad1) -> VCCD_mon
- R26 pad 2: unconnected-(R26-Pad2) -> GND
- R27 pad 1: unconnected-(R27-Pad1) -> VCCD_mon
- R27 pad 2: unconnected-(R27-Pad2) -> VDD
- R28 pad 1: unconnected-(R28-Pad1) -> Net-(U6-Pad1)
- R28 pad 2: unconnected-(R28-Pad2) -> Net-(U4-Pad6)
- R29 pad 1: unconnected-(R29-Pad1) -> Net-(R29-Pad1)
- R29 pad 2: unconnected-(R29-Pad2) -> Net-(C23-Pad1)
- R3 pad 1: unconnected-(R3-Pad1) -> Net-(U1-Pad31)
- R3 pad 2: unconnected-(R3-Pad2) -> UART_RX
- R30 pad 1: unconnected-(R30-Pad1) -> Net-(U6-Pad1)
- R30 pad 2: unconnected-(R30-Pad2) -> Net-(R32-Pad1)
- R31 pad 1: unconnected-(R31-Pad1) -> Net-(R31-Pad1)
- R31 pad 2: unconnected-(R31-Pad2) -> Net-(R31-Pad2)
- R32 pad 1: unconnected-(R32-Pad1) -> Net-(R32-Pad1)
- R32 pad 2: unconnected-(R32-Pad2) -> Net-(C33-Pad2)
- R33 pad 1: unconnected-(R33-Pad1) -> Net-(R33-Pad1)
- R33 pad 2: unconnected-(R33-Pad2) -> Net-(R32-Pad1)
- R34 pad 1: unconnected-(R34-Pad1) -> Pullup
- R34 pad 2: unconnected-(R34-Pad2) -> GND
- R4 pad 1: unconnected-(R4-Pad1) -> CS_Pressure
- R4 pad 2: unconnected-(R4-Pad2) -> Net-(R4-Pad2)
- R5 pad 1: unconnected-(R5-Pad1) -> Net-(R5-Pad1)
- R5 pad 2: unconnected-(R5-Pad2) -> NRST
- R6 pad 1: unconnected-(R6-Pad1) -> Net-(U1-Pad20)
- R6 pad 2: unconnected-(R6-Pad2) -> CS_EEPROM
- R7 pad 1: unconnected-(R7-Pad1) -> Net-(R7-Pad1)
- R7 pad 2: unconnected-(R7-Pad2) -> Out
- R8 pad 1: unconnected-(R8-Pad1) -> Out
- R8 pad 2: unconnected-(R8-Pad2) -> Net-(R33-Pad1)
- R9 pad 1: unconnected-(R9-Pad1) -> GND
- R9 pad 2: unconnected-(R9-Pad2) -> VCCA_mon
- SH1 pad 1: unconnected-(SH1-Pad1) -> GND
- U1 pad 1: unconnected-(U1-Pad1) -> VDD
- U1 pad 10: unconnected-(U1-Pad10) -> Net-(U1-Pad20)
- U1 pad 11: unconnected-(U1-Pad11) -> Net-(R7-Pad1)
- U1 pad 15: unconnected-(U1-Pad15) -> Net-(U1-Pad15)
- U1 pad 16: unconnected-(U1-Pad16) -> Net-(U1-Pad16)
- U1 pad 17: unconnected-(U1-Pad17) -> Net-(U1-Pad17)
- U1 pad 18: unconnected-(U1-Pad18) -> VCCA_mon
- U1 pad 19: unconnected-(U1-Pad19) -> Net-(R14-Pad2)
- U1 pad 20: unconnected-(U1-Pad20) -> Net-(U1-Pad20)
- U1 pad 22: unconnected-(U1-Pad22) -> Net-(U1-Pad22)
- U1 pad 23: unconnected-(U1-Pad23) -> GND
- U1 pad 24: unconnected-(U1-Pad24) -> VDD
- U1 pad 25: unconnected-(U1-Pad25) -> Net-(U1-Pad25)
- U1 pad 30: unconnected-(U1-Pad30) -> Net-(U1-Pad30)
- U1 pad 31: unconnected-(U1-Pad31) -> Net-(U1-Pad31)
- U1 pad 34: unconnected-(U1-Pad34) -> Net-(U1-Pad34)
- U1 pad 35: unconnected-(U1-Pad35) -> GND
- U1 pad 36: unconnected-(U1-Pad36) -> VDD
- U1 pad 37: unconnected-(U1-Pad37) -> Net-(U1-Pad37)
- U1 pad 39: unconnected-(U1-Pad39) -> Net-(R20-Pad2)
- U1 pad 41: unconnected-(U1-Pad41) -> Net-(U1-Pad41)
- U1 pad 42: unconnected-(U1-Pad42) -> Net-(U1-Pad42)
- U1 pad 47: unconnected-(U1-Pad47) -> GND
- U1 pad 48: unconnected-(U1-Pad48) -> VDD
- U1 pad 5: unconnected-(U1-Pad5) -> Net-(R4-Pad2)
- U1 pad 7: unconnected-(U1-Pad7) -> Net-(R5-Pad1)
- U1 pad 8: unconnected-(U1-Pad8) -> GND
- U1 pad 9: unconnected-(U1-Pad9) -> VDD
- U2 pad 1: unconnected-(U2-Pad1) -> Switch_1
- U2 pad 2: unconnected-(U2-Pad2) -> VCC
- U2 pad 3: unconnected-(U2-Pad3) -> GND
- U2 pad 4: unconnected-(U2-Pad4) -> GND
- U2 pad 5: unconnected-(U2-Pad5) -> Net-(U2-Pad5)
- U2 pad 6: unconnected-(U2-Pad6) -> Net-(U4-Pad6)
- U3 pad 1: unconnected-(U3-Pad1) -> Switch_2
- U3 pad 2: unconnected-(U3-Pad2) -> VCC
- U3 pad 3: unconnected-(U3-Pad3) -> GND
- U3 pad 4: unconnected-(U3-Pad4) -> GND
- U3 pad 6: unconnected-(U3-Pad6) -> Net-(U4-Pad6)
- U4 pad 1: unconnected-(U4-Pad1) -> Switch_3
- U4 pad 2: unconnected-(U4-Pad2) -> VCC
- U4 pad 3: unconnected-(U4-Pad3) -> GND
- U4 pad 4: unconnected-(U4-Pad4) -> GND
- U4 pad 5: unconnected-(U4-Pad5) -> Net-(U4-Pad5)
- U4 pad 6: unconnected-(U4-Pad6) -> Net-(U4-Pad6)
- U5 pad 1: unconnected-(U5-Pad1) -> Net-(C33-Pad2)
- U5 pad 2: unconnected-(U5-Pad2) -> Net-(R29-Pad1)
- U5 pad 3: unconnected-(U5-Pad3) -> Net-(R29-Pad1)
- U5 pad 5: unconnected-(U5-Pad5) -> Net-(U4-Pad6)
- U5 pad 6: unconnected-(U5-Pad6) -> Net-(R31-Pad2)
- U5 pad 7: unconnected-(U5-Pad7) -> Net-(R31-Pad2)
- U6 pad 1: unconnected-(U6-Pad1) -> Net-(U6-Pad1)
- U6 pad 2: unconnected-(U6-Pad2) -> GND
- U6 pad 4: unconnected-(U6-Pad4) -> Net-(R32-Pad1)
- U7 pad 1: unconnected-(U7-Pad1) -> +3V8
- U7 pad 2: unconnected-(U7-Pad2) -> GND
- U7 pad 3: unconnected-(U7-Pad3) -> +3V8
- U7 pad 4: unconnected-(U7-Pad4) -> Net-(U7-Pad4)
- U7 pad 5: unconnected-(U7-Pad5) -> Net-(U7-Pad5)
